Commit message: Editato limite basso

File: custom_robotiq_description/urdf/robotiq_2f_140.xacro (robot description, xacro)
@@ -150,5 +150,6 @@
       <child link="${prefix}left_outer_knuckle" />
       <axis xyz="-1 0 0" />
-      <limit lower="-0.07" upper="0.7" velocity="2.0" effort="1000" /> // edited lower limit
+      <!-- Edited lower limit to -0.07 -->
+      <limit lower="-0.07" upper="0.7" velocity="2.0" effort="1000" />
     </joint>
     <xacro:finger_joints prefix="${prefix}" fingerprefix="left" reflect="1.0"/>

File: custom_robotiq_description/urdf/robotiq_2f_140_macro.urdf.xacro (robot description, xacro)
@@ -73,5 +73,5 @@
       </joint>
       <!-- Include the finger xacros and run them -->
-      <xacro:include filename="$(find robotiq_description)/urdf/robotiq_2f_140.xacro" />
+      <xacro:include filename="$(find custom_robotiq_description)/urdf/robotiq_2f_140.xacro" />
       <xacro:finger_links prefix="${prefix}" fingerprefix="left" stroke="140"/>
       <xacro:finger_links prefix="${prefix}" fingerprefix="right" stroke="140"/>
